File: Плата обмоток/Плата обмоток.kicad_sch (KiCad schematic)
At the start: 22 parts, among them J1 4900, J10 4900, J11 4900, J12 4900, J13 4900, J14 A1, J15 A2, J16 B1, J17 B2, J18 C1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

Commit message: Добавил все документы
Other:
- title: (none) -> Соединительная плата ЭЛП
- moved on the sheet: J1, J10, J11, J12, J13, J14, J15, J16, J17, J18, J19, J2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
