File: Плата обмоток/Плата обмоток.kicad_sch (KiCad schematic)
At the start: 7 parts, among them J1 A_OUT, J1 B_OUT, J1 C_OUT, J4 Conn_01x02, J6 Conn_01x02, J7 Conn_01x02, J8 Conn_02x02_Odd_Even

Commit message: Добавил ножевые разъёмы
Parts:
- removed J1: A_OUT, Connector_My:Power_Wire, symbol Connector_Generic:Conn_01x01
- removed J1: C_OUT, Connector_My:Power_Wire, symbol Connector_Generic:Conn_01x01
- removed J1: B_OUT, Connector_My:Power_Wire, symbol Connector_Generic:Conn_01x01
- added J1, J10, J11, J12, J13, J2, J3, J8, J9: 4900, Connector_My:3551, symbol 4900:4900
Connections:
- net A_OUT: now also J1.1, J1.2, J2.1, J2.2, J3.1, J3.2
- net B_OUT: now also J10.1, J10.2, J8.1, J8.2, J9.1, J9.2
- net C_OUT: now also J11.1, J11.2, J12.1, J12.2, J13.1, J13.2

Commit message: Прямой вывод обмоток на плату
Parts:
- added H1: MountingHole, MountingHole:MountingHole_2.1mm, symbol Mechanical:MountingHole
Changed lines of the file:
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@@
+    )
+  )
+  (symbol (lib_id "Mechanical:MountingHole") (at 193.04 72.39 0) (unit 1)
+    (in_bom yes) (on_board yes) (dnp no) (fields_autoplaced)
+    (property "Reference" "H1" (at 195.58 71.755 0)
+      (effects (font (size 1.27 1.27)) (justify left))
+    )
+    (property "Value" "MountingHole" (at 195.58 74.295 0)
+      (effects (font (size 1.27 1.27)) (justify left))
+    )
+    (property "Footprint" "MountingHole:MountingHole_2.1mm" (at 193.04 72.39 0)
+      (effects (font (size 1.27 1.27)) hide)
+    )
+    (property "Datasheet" "~" (at 193.04 72.39 0)
+      (effects (font (size 1.27 1.27)) hide)
+    )
+    (instances
+      (project "Плата обмоток"
+        (path "/7abc0ce6-258d-434e-9c1a-83bc5738d31c"
+          (reference "H1") (unit 1)
+        )
+      )
     )
   )

Commit message: Расставил ножевые разъёмы финально
Parts:
- added J14: A1, Connector_My:Coil, symbol Connector:Conn_01x01_Pin
- added J15: A2, Connector_My:Coil, symbol Connector:Conn_01x01_Pin
- added J16: B1, Connector_My:Coil, symbol Connector:Conn_01x01_Pin
- added J17: B2, Connector_My:Coil, symbol Connector:Conn_01x01_Pin
- added J18: C1, Connector_My:Coil, symbol Connector:Conn_01x01_Pin
- added J19: C2, Connector_My:Coil, symbol Connector:Conn_01x01_Pin
Connections:
- net A_OUT: now also J15.1 (Pin_1), J16.1 (Pin_1)
- net B_OUT: now also J17.1 (Pin_1), J18.1 (Pin_1)
- net C_OUT: now also J14.1 (Pin_1), J19.1 (Pin_1)
Changed lines of the file:
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@@
   (junction (at 99.06 123.19) (diameter 0) (color 0 0 0 0)
   )
+  (junction (at 234.95 80.01) (diameter 0) (color 0 0 0 0)
+  )
+  (junction (at 234.95 58.42) (diameter 0) (color 0 0 0 0)
+  )
   (junction (at 64.77 116.84) (diameter 0) (color 0 0 0 0)
   )
@@
   (junction (at 99.06 116.84) (diameter 0) (color 0 0 0 0)
   )
+  (junction (at 234.95 69.85) (diameter 0) (color 0 0 0 0)
+  )
   (junction (at 64.77 114.3) (diameter 0) (color 0 0 0 0)
   )
@@
     (stroke (width 0) (type default))
   )
+  (wire (pts (xy 232.41 82.55) (xy 234.95 82.55))
+    (stroke (width 0) (type default))
+  )
   (wire (pts (xy 66.04 105.41) (xy 64.77 105.41))
     (stroke (width 0) (type default))
   )
+  (wire (pts (xy 234.95 55.88) (xy 234.95 58.42))
+    (stroke (width 0) (type default))
+  )
   (wire (pts (xy 133.35 107.95) (xy 134.62 107.95))
     (stroke (width 0) (type default))
   )
+  (wire (pts (xy 234.95 80.01) (xy 234.95 77.47))
+    (stroke (width 0) (type default))
+  )
   (wire (pts (xy 64.77 123.19) (xy 64.77 125.73))
     (stroke (width 0) (type default))
@@
     (stroke (width 0) (type default))
   )
+  (wire (pts (xy 232.41 67.31) (xy 234.95 67.31))
+    (stroke (width 0) (type default))
+  )
+  (wire (pts (xy 234.95 67.31) (xy 234.95 69.85))
+    (stroke (width 0) (type default))
+  )
+  (wire (pts (xy 234.95 77.47) (xy 232.41 77.47))
+    (stroke (width 0) (type default))
+  )
   (wire (pts (xy 99.06 114.3) (xy 100.33 114.3))
     (stroke (width 0) (type default))
@@
     (stroke (width 0) (type default))
   )
+  (wire (pts (xy 234.95 69.85) (xy 234.95 72.39))
+    (stroke (width 0) (type default))
+  )
   (wire (pts (xy 64.77 116.84) (xy 66.04 116.84))
     (stroke (width 0) (type default))
@@
     (stroke (width 0) (type default))
   )
+  (wire (pts (xy 234.95 58.42) (xy 236.22 58.42))
+    (stroke (width 0) (type default))
+  )
   (wire (pts (xy 133.35 123.19) (xy 133.35 125.73))
     (stroke (width 0) (type default))
@@
     (stroke (width 0) (type default))
   )
+  (wire (pts (xy 232.41 55.88) (xy 234.95 55.88))
+    (stroke (width 0) (type default))
+  )
+  (wire (pts (xy 234.95 69.85) (xy 236.22 69.85))
+    (stroke (width 0) (type default))
+  )
   (wire (pts (xy 64.77 125.73) (xy 66.04 125.73))
     (stroke (width 0) (type default))
@@
     (stroke (width 0) (type default))
   )
+  (wire (pts (xy 234.95 82.55) (xy 234.95 80.01))
+    (stroke (width 0) (type default))
+  )
   (wire (pts (xy 99.06 123.19) (xy 100.33 123.19))
     (stroke (width 0) (type default))
   )
+  (wire (pts (xy 232.41 60.96) (xy 234.95 60.96))
+    (stroke (width 0) (type default))
+  )
+  (wire (pts (xy 234.95 80.01) (xy 236.22 80.01))
+    (stroke (width 0) (type default))
+  )
   (wire (pts (xy 64.77 107.95) (xy 64.77 114.3))
     (stroke (width 0) (type default))
@@
   )
   (wire (pts (xy 64.77 105.41) (xy 64.77 107.95))
+    (stroke (width 0) (type default))
+  )
+  (wire (pts (xy 234.95 72.39) (xy 232.41 72.39))
+    (stroke (width 0) (type default))
+  )
+  (wire (pts (xy 234.95 58.42) (xy 234.95 60.96))
     (stroke (width 0) (type default))
   )
@@
     )
   )
+  (global_label "C_OUT" (shape input) (at 236.22 58.42 0) (fields_autoplaced)
+    (effects (font (size 1.27 1.27)) (justify left))
+    (property "Intersheetrefs" "${INTERSHEET_REFS}" (at 244.992 58.42 0)
+      (effects (font (size 1.27 1.27)) (justify left) hide)
+    )
+  )
   (global_label "PTC_Coil_C" (shape input) (at 140.97 85.09 180) (fields_autoplaced)
     (effects (font (size 1.27 1.27)) (justify right))
@@
     )
   )
+  (global_label "A_OUT" (shape input) (at 236.22 80.01 0) (fields_autoplaced)
+    (effects (font (size 1.27 1.27)) (justify left))
+    (property "Intersheetrefs" "${INTERSHEET_REFS}" (at 244.8106 80.01 0)
+      (effects (font (size 1.27 1.27)) (justify left) hide)
+    )
+  )
   (global_label "A_OUT" (shape input) (at 62.23 115.57 180) (fields_autoplaced)
     (effects (font (size 1.27 1.27)) (justify right))
@@
     )
   )
+  (global_label "B_OUT" (shape input) (at 236.22 69.85 0) (fields_autoplaced)
+    (effects (font (size 1.27 1.27)) (justify left))
+    (property "Intersheetrefs" "${INTERSHEET_REFS}" (at 244.992 69.85 0)
+      (effects (font (size 1.27 1.27)) (justify left) hide)
+    )
+  )
+  (symbol (lib_id "Connector:Conn_01x01_Pin") (at 227.33 60.96 0) (unit 1)
+    (in_bom yes) (on_board yes) (dnp no) (fields_autoplaced)
+    (property "Reference" "J14" (at 227.965 57.15 0)
+      (effects (font (size 1.27 1.27)))
+    )
+    (property "Value" "A1" (at 227.965 59.69 0)
+      (effects (font (size 1.27 1.27)))
+    )
+    (property "Footprint" "Connector_My:Coil" (at 227.33 60.96 0)
+      (effects (font (size 1.27 1.27)) hide)
+    )
+    (property "Datasheet" "~" (at 227.33 60.96 0)
+      (effects (font (size 1.27 1.27)) hide)
+    )
+    (pin "1")
+    (instances
+      (project "Плата обмоток"
+        (path "/7abc0ce6-258d-434e-9c1a-83bc5738d31c"
+          (reference "J14") (unit 1)
+        )
+      )
+    )
+  )
   (symbol (lib_id "4900:4900") (at 134.62 105.41 0) (unit 1)
     (in_bom yes) (on_board yes) (dnp no) (fields_autoplaced)
@@
         (path "/7abc0ce6-258d-434e-9c1a-83bc5738d31c"
           (reference "J11") (unit 1)
+        )
+      )
+    )
+  )
+  (symbol (lib_id "Connector:Conn_01x01_Pin") (at 227.33 72.39 0) (unit 1)
+    (in_bom yes) (on_board yes) (dnp no) (fields_autoplaced)
+    (property "Reference" "J18" (at 227.965 68.58 0)
+      (effects (font (size 1.27 1.27)))
+    )
+    (property "Value" "C1" (at 227.965 71.12 0)
+      (effects (font (size 1.27 1.27)))
+    )
+    (property "Footprint" "Connector_My:Coil" (at 227.33 72.39 0)
+      (effects (font (size 1.27 1.27)) hide)
+    )
+    (property "Datasheet" "~" (at 227.33 72.39 0)
+      (effects (font (size 1.27 1.27)) hide)
+    )
+    (pin "1")
+    (instances
+      (project "Плата обмоток"
+        (path "/7abc0ce6-258d-434e-9c1a-83bc5738d31c"
+          (reference "J18") (unit 1)
         )
       )
@@
     )
   )
+  (symbol (lib_id "Connector:Conn_01x01_Pin") (at 227.33 77.47 0) (unit 1)
+    (in_bom yes) (on_board yes) (dnp no) (fields_autoplaced)
+    (property "Reference" "J15" (at 227.965 73.66 0)
+      (effects (font (size 1.27 1.27)))
+    )
+    (property "Value" "A2" (at 227.965 76.2 0)
+      (effects (font (size 1.27 1.27)))
+    )
+    (property "Footprint" "Connector_My:Coil" (at 227.33 77.47 0)
+      (effects (font (size 1.27 1.27)) hide)
+    )
+    (property "Datasheet" "~" (at 227.33 77.47 0)
+      (effects (font (size 1.27 1.27)) hide)
+    )
+    (pin "1")
+    (instances
+      (project "Плата обмоток"
+        (path "/7abc0ce6-258d-434e-9c1a-83bc5738d31c"
+          (reference "J15") (unit 1)
+        )
+      )
+    )
+  )
   (symbol (lib_id "4900:4900") (at 66.04 105.41 0) (unit 1)
     (in_bom yes) (on_board yes) (dnp no) (fields_autoplaced)
@@
         (path "/7abc0ce6-258d-434e-9c1a-83bc5738d31c"
           (reference "J1") (unit 1)
+        )
+      )
+    )
+  )
+  (symbol (lib_id "Connector:Conn_01x01_Pin") (at 227.33 67.31 0) (unit 1)
+    (in_bom yes) (on_board yes) (dnp no) (fields_autoplaced)
+    (property "Reference" "J17" (at 227.965 63.5 0)
+      (effects (font (size 1.27 1.27)))
+    )
+    (property "Value" "B2" (at 227.965 66.04 0)
+      (effects (font (size 1.27 1.27)))
+    )
+    (property "Footprint" "Connector_My:Coil" (at 227.33 67.31 0)
+      (effects (font (size 1.27 1.27)) hide)
+    )
+    (property "Datasheet" "~" (at 227.33 67.31 0)
+      (effects (font (size 1.27 1.27)) hide)
+    )
+    (pin "1")
+    (instances
+      (project "Плата обмоток"
+        (path "/7abc0ce6-258d-434e-9c1a-83bc5738d31c"
+          (reference "J17") (unit 1)
         )
       )
@@
     )
   )
+  (symbol (lib_id "Connector:Conn_01x01_Pin") (at 227.33 55.88 0) (unit 1)
+    (in_bom yes) (on_board yes) (dnp no)
+    (property "Reference" "J19" (at 227.965 52.07 0)
+      (effects (font (size 1.27 1.27)))
+    )
+    (property "Value" "C2" (at 227.965 54.61 0)
+      (effects (font (size 1.27 1.27)))
+    )
+    (property "Footprint" "Connector_My:Coil" (at 227.33 55.88 0)
+      (effects (font (size 1.27 1.27)) hide)
+    )
+    (property "Datasheet" "~" (at 227.33 55.88 0)
+      (effects (font (size 1.27 1.27)) hide)
+    )
+    (pin "1")
+    (instances
+      (project "Плата обмоток"
+        (path "/7abc0ce6-258d-434e-9c1a-83bc5738d31c"
+          (reference "J19") (unit 1)
+        )
+      )
+    )
+  )
   (symbol (lib_id "4900:4900") (at 66.04 123.19 0) (unit 1)
     (in_bom yes) (on_board yes) (dnp no) (fields_autoplaced)
@@
         )
       )
+    )
+  )
+  (symbol (lib_id "Connector:Conn_01x01_Pin") (at 227.33 82.55 0) (unit 1)
+    (in_bom yes) (on_board yes) (dnp no) (fields_autoplaced)
+    (property "Reference" "J16" (at 227.965 78.74 0)
+      (effects (font (size 1.27 1.27)))
+    )
+    (property "Value" "B1" (at 227.965 81.28 0)
+      (effects (font (size 1.27 1.27)))
+    )
+    (property "Footprint" "Connector_My:Coil" (at 227.33 82.55 0)
+      (effects (font (size 1.27 1.27)) hide)
+    )
+    (property "Datasheet" "~" (at 227.33 82.55 0)
+      (effects (font (size 1.27 1.27)) hide)
+    )
+    (pin "1")
+    (instances
+      (project "Плата обмоток"
+        (path "/7abc0ce6-258d-434e-9c1a-83bc5738d31c"
+          (reference "J16") (unit 1)
+        )
+      )

Commit message: Ещё доработать
Parts:
- added H2, H3, H4: MountingHole, MountingHole:MountingHole_3.2mm_M3, symbol Mechanical:MountingHole
Connections:
- net B_OUT: now also J11.1, J11.2, J12.1, J12.2, J13.1, J13.2; no longer J10.1, J10.2, J8.1, J8.2, J9.1, J9.2
- net C_OUT: now also J10.1, J10.2, J8.1, J8.2, J9.1, J9.2; no longer J11.1, J11.2, J12.1, J12.2, J13.1, J13.2
Changed lines of the file:
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@@
     (stroke (width 0) (type default))
   )
-  (global_label "C_OUT" (shape input) (at 130.81 115.57 180) (fields_autoplaced)
+  (global_label "C_OUT" (shape input) (at 96.52 115.57 180) (fields_autoplaced)
     (effects (font (size 1.27 1.27)) (justify right))
-    (property "Intersheetrefs" "${INTERSHEET_REFS}" (at 121.9586 115.57 0)
+    (property "Intersheetrefs" "${INTERSHEET_REFS}" (at 87.6686 115.57 0)
       (effects (font (size 1.27 1.27)) (justify right) hide)
     )
@@
     )
   )
-  (global_label "B_OUT" (shape input) (at 96.52 115.57 180) (fields_autoplaced)
+  (global_label "B_OUT" (shape input) (at 130.81 115.57 180) (fields_autoplaced)
     (effects (font (size 1.27 1.27)) (justify right))
-    (property "Intersheetrefs" "${INTERSHEET_REFS}" (at 87.6686 115.57 0)
+    (property "Intersheetrefs" "${INTERSHEET_REFS}" (at 121.9586 115.57 0)
       (effects (font (size 1.27 1.27)) (justify right) hide)
     )
@@
     )
   )
+  (symbol (lib_id "Mechanical:MountingHole") (at 193.04 90.17 0) (unit 1)
+    (in_bom yes) (on_board yes) (dnp no) (fields_autoplaced)
+    (property "Reference" "H4" (at 195.58 89.535 0)
+      (effects (font (size 1.27 1.27)) (justify left) hide)
+    )
+    (property "Value" "MountingHole" (at 195.58 92.075 0)
+      (effects (font (size 1.27 1.27)) (justify left) hide)
+    )
+    (property "Footprint" "MountingHole:MountingHole_3.2mm_M3" (at 193.04 90.17 0)
+      (effects (font (size 1.27 1.27)) hide)
+    )
+    (property "Datasheet" "~" (at 193.04 90.17 0)
+      (effects (font (size 1.27 1.27)) hide)
+    )
+    (instances
+      (project "Плата обмоток"
+        (path "/7abc0ce6-258d-434e-9c1a-83bc5738d31c"
+          (reference "H4") (unit 1)
+        )
+      )
+    )
+  )
   (symbol (lib_id "4900:4900") (at 100.33 105.41 0) (unit 1)
     (in_bom yes) (on_board yes) (dnp no) (fields_autoplaced)
@@
     )
   )
+  (symbol (lib_id "Mechanical:MountingHole") (at 193.04 85.09 0) (unit 1)
+    (in_bom yes) (on_board yes) (dnp no) (fields_autoplaced)
+    (property "Reference" "H3" (at 195.58 84.455 0)
+      (effects (font (size 1.27 1.27)) (justify left) hide)
+    )
+    (property "Value" "MountingHole" (at 195.58 86.995 0)
+      (effects (font (size 1.27 1.27)) (justify left) hide)
+    )
+    (property "Footprint" "MountingHole:MountingHole_3.2mm_M3" (at 193.04 85.09 0)
+      (effects (font (size 1.27 1.27)) hide)
+    )
+    (property "Datasheet" "~" (at 193.04 85.09 0)
+      (effects (font (size 1.27 1.27)) hide)
+    )
+    (instances
+      (project "Плата обмоток"
+        (path "/7abc0ce6-258d-434e-9c1a-83bc5738d31c"
+          (reference "H3") (unit 1)
+        )
+      )
+    )
+  )
   (symbol (lib_id "Connector_Generic:Conn_02x02_Odd_Even") (at 180.34 44.45 0) (unit 1)
     (in_bom yes) (on_board yes) (dnp no) (fields_autoplaced)
@@
         )
       )
+    )
+  )
+  (symbol (lib_id "Mechanical:MountingHole") (at 193.04 80.01 0) (unit 1)
+    (in_bom yes) (on_board yes) (dnp no) (fields_autoplaced)
+    (property "Reference" "H2" (at 195.58 79.375 0)
+      (effects (font (size 1.27 1.27)) (justify left) hide)
+    )
+    (property "Value" "MountingHole" (at 195.58 81.915 0)
+      (effects (font (size 1.27 1.27)) (justify left) hide)
+    )
+    (property "Footprint" "MountingHole:MountingHole_3.2mm_M3" (at 193.04 80.01 0)
+      (effects (font (size 1.27 1.27)) hide)
+    )
+    (property "Datasheet" "~" (at 193.04 80.01 0)
+      (effects (font (size 1.27 1.27)) hide)
+    )
+    (instances
+      (project "Плата обмоток"
+        (path "/7abc0ce6-258d-434e-9c1a-83bc5738d31c"
+          (reference "H2") (unit 1)
+        )
+      )

Commit message: Собираю документацию
Parts:
- removed H1: MountingHole, MountingHole:MountingHole_2.1mm, symbol Mechanical:MountingHole
- J4, J6, J7: footprint Connector_PinHeader_2.54mm:PinHeader_1x02_P2.54mm_Vertical -> Connector_Molex:Molex_PicoBlade_53048-0210_1x02_P1.25mm_Horizontal
Connections:
- net GNDA: now also J8.2 (Pin_2); no longer J8.4 (Pin_4)
- net PTC_Coil_B: now also J8.4 (Pin_4); no longer J8.3 (Pin_3)
- net PTC_Coil_C: now also J8.3 (Pin_3); no longer J8.2 (Pin_2)
Changed lines of the file:
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@@
     )
   )
-  (global_label "PTC_Coil_B" (shape input) (at 175.26 46.99 180) (fields_autoplaced)
-    (effects (font (size 1.27 1.27)) (justify right))
-    (property "Intersheetrefs" "${INTERSHEET_REFS}" (at 161.873 46.99 0)
-      (effects (font (size 1.27 1.27)) (justify right) hide)
+  (global_label "PTC_Coil_B" (shape input) (at 187.96 46.99 0) (fields_autoplaced)
+    (effects (font (size 1.27 1.27)) (justify left))
+    (property "Intersheetrefs" "${INTERSHEET_REFS}" (at 201.347 46.99 0)
+      (effects (font (size 1.27 1.27)) (justify left) hide)
     )
   )
@@
     )
   )
-  (global_label "PTC_Coil_C" (shape input) (at 187.96 44.45 0) (fields_autoplaced)
-    (effects (font (size 1.27 1.27)) (justify left))
-    (property "Intersheetrefs" "${INTERSHEET_REFS}" (at 201.347 44.45 0)
-      (effects (font (size 1.27 1.27)) (justify left) hide)
+  (global_label "PTC_Coil_C" (shape input) (at 175.26 46.99 180) (fields_autoplaced)
+    (effects (font (size 1.27 1.27)) (justify right))
+    (property "Intersheetrefs" "${INTERSHEET_REFS}" (at 161.873 46.99 0)
+      (effects (font (size 1.27 1.27)) (justify right) hide)
     )
   )
@@
       (effects (font (size 1.27 1.27)) (justify left))
     )
-    (property "Footprint" "Connector_PinHeader_2.54mm:PinHeader_1x02_P2.54mm_Vertical" (at 146.05 69.85 0)
+    (property "Footprint" "Connector_Molex:Molex_PicoBlade_53048-0210_1x02_P1.25mm_Horizontal" (at 146.05 69.85 0)
       (effects (font (size 1.27 1.27)) hide)
     )
@@
       (effects (font (size 1.27 1.27)) (justify left))
     )
-    (property "Footprint" "Connector_PinHeader_2.54mm:PinHeader_1x02_P2.54mm_Vertical" (at 146.05 77.47 0)
+    (property "Footprint" "Connector_Molex:Molex_PicoBlade_53048-0210_1x02_P1.25mm_Horizontal" (at 146.05 77.47 0)
       (effects (font (size 1.27 1.27)) hide)
     )
@@
       (effects (font (size 1.27 1.27)) (justify left))
     )
-    (property "Footprint" "Connector_PinHeader_2.54mm:PinHeader_1x02_P2.54mm_Vertical" (at 146.05 85.09 0)
+    (property "Footprint" "Connector_Molex:Molex_PicoBlade_53048-0210_1x02_P1.25mm_Horizontal" (at 146.05 85.09 0)
       (effects (font (size 1.27 1.27)) hide)
     )
@@
     )
   )
-  (symbol (lib_id "power:GNDA") (at 187.96 46.99 90) (unit 1)
-    (in_bom yes) (on_board yes) (dnp no) (fields_autoplaced)
-    (property "Reference" "#PWR038" (at 194.31 46.99 0)
-      (effects (font (size 1.27 1.27)) hide)
-    )
-    (property "Value" "GNDA" (at 191.77 46.99 90)
+  (symbol (lib_id "power:GNDA") (at 187.96 44.45 90) (unit 1)
+    (in_bom yes) (on_board yes) (dnp no) (fields_autoplaced)
+    (property "Reference" "#PWR038" (at 194.31 44.45 0)
+      (effects (font (size 1.27 1.27)) hide)
+    )
+    (property "Value" "GNDA" (at 191.77 44.45 90)
       (effects (font (size 1.27 1.27)) (justify right))
     )
-    (property "Footprint" "" (at 187.96 46.99 0)
-      (effects (font (size 1.27 1.27)) hide)
-    )
-    (property "Datasheet" "" (at 187.96 46.99 0)
+    (property "Footprint" "" (at 187.96 44.45 0)
+      (effects (font (size 1.27 1.27)) hide)
+    )
+    (property "Datasheet" "" (at 187.96 44.45 0)
       (effects (font (size 1.27 1.27)) hide)
     )
@@
         )
       )
-    )
-  )
-  (symbol (lib_id "Mechanical:MountingHole") (at 193.04 72.39 0) (unit 1)
-    (in_bom yes) (on_board yes) (dnp no) (fields_autoplaced)
-    (property "Reference" "H1" (at 195.58 71.755 0)
-      (effects (font (size 1.27 1.27)) (justify left))
-    )
-    (property "Value" "MountingHole" (at 195.58 74.295 0)
-      (effects (font (size 1.27 1.27)) (justify left))
-    )
-    (property "Footprint" "MountingHole:MountingHole_2.1mm" (at 193.04 72.39 0)
-      (effects (font (size 1.27 1.27)) hide)
-    )
-    (property "Datasheet" "~" (at 193.04 72.39 0)
-      (effects (font (size 1.27 1.27)) hide)
-    )
-    (instances
-      (project "Плата обмоток"
-        (path "/7abc0ce6-258d-434e-9c1a-83bc5738d31c"
-          (reference "H1") (unit 1)
-        )
-      )

Commit message: Версия под отчётность
Parts:
- removed H2, H3, H4: MountingHole, MountingHole:MountingHole_3.2mm_M3, symbol Mechanical:MountingHole
- removed J1, J10, J11, J12, J13, J2, J3, J8, J9: 4900, Connector_My:3551, symbol 4900:4900
- removed J14: A1, Connector_My:Coil, symbol Connector:Conn_01x01_Pin
- removed J15: A2, Connector_My:Coil, symbol Connector:Conn_01x01_Pin
- removed J16: B1, Connector_My:Coil, symbol Connector:Conn_01x01_Pin
- removed J17: B2, Connector_My:Coil, symbol Connector:Conn_01x01_Pin
- removed J18: C1, Connector_My:Coil, symbol Connector:Conn_01x01_Pin
- removed J19: C2, Connector_My:Coil, symbol Connector:Conn_01x01_Pin
- removed J4, J6, J7: Conn_01x02, Connector_Molex:Molex_PicoBlade_53048-0210_1x02_P1.25mm_Horizontal, symbol Connector_Generic:Conn_01x02
- removed J8: Conn_02x02_Odd_Even, Connector_PinSocket_2.54mm:PinSocket_2x02_P2.54mm_Vertical, symbol Connector_Generic:Conn_02x02_Odd_Even
Other:
- added sheet Connection List (Connection List.kicad_sch)
- added sheet Connectors (Connectors.kicad_sch)
- note added: "Схема электрическая"
- note added: "принципиальная"
- company: (none) -> Московский Политех
- title: (none) -> Узел соединительный
