File: Плата обмоток/Плата обмоток.kicad_pcb (KiCad board)
At the start: 4 copper layers, 58 x 58 mm, 24 parts, among them J1 4900, J10 4900, J11 4900, J12 4900, J13 4900, J14 Conn_01x03, J15 C1, J16 4900, J17 A2, J18 B1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

Commit message: Базовый вариант с пайкой
Parts:
- moved J15 4.96 mm to (147.0, 46.2)
- moved J7 4.51 mm to (152.0, 46.2)
Other:
- outline, holes or cut-outs redrawn
Changed lines of the file:
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@@
   )
   (footprint "Connector_My:Coil" (layer "B.Cu")
-    (at 156.464 46.228 180)
+    (at 151.950502 46.228 180)
     (property "Sheetfile" "Connectors.kicad_sch")
     (property "Sheetname" "Connectors")
@@
     (pad "1" thru_hole circle (at 0 0 180) (size 4 4) (drill 2) (layers "*.Cu" "*.Mask")
       (net 5 "B") (pinfunction "Pin_1") (pintype "passive"))
+    (model "C:/Users/alexa/Desktop/Проекты/КАМАЗ/Плата обмоток/KAMAZ_Coil_PCB/3D модели/KF2-M3-ET.stp"
+      (offset (xyz 0 0 -3.25))
+      (scale (xyz 1 1 1))
+      (rotate (xyz 0 -90 0))
+    )
   )
   (footprint "Connector_PinSocket_2.54mm:PinSocket_1x03_P2.54mm_Vertical" (layer "B.Cu")
@@
   )
   (footprint "Connector_My:Coil" (layer "B.Cu")
-    (at 141.986 46.228 180)
+    (at 146.950502 46.228 180)
     (property "Sheetfile" "Connectors.kicad_sch")
     (property "Sheetname" "Connectors")
@@
   (gr_circle (center 149.450502 71.074296) (end 178.450502 71.074296)
     (stroke (width 0.15) (type default)) (fill none) (layer "Edge.Cuts"))
-  (gr_circle (center 149.450502 71.074296) (end 167.374477 71.074296)
+  (gr_circle (center 149.450502 71.074296) (end 158.450502 71.074296)
     (stroke (width 0.1) (type default)) (fill none) (layer "Edge.Cuts"))
   (gr_text "" (at -48.324542 258.222 90) (layer "Dwgs.User")
@@
       (pts
         (xy 180.975 99.06)
-        (xy 159.385 99.06)
-        (xy 159.385 61.595)
+        (xy 155.321 99.06)
+        (xy 155.321 61.595)
         (xy 180.34 61.595)
       )
@@
       (pts
         (xy 118.11 99.06)
-        (xy 139.7 99.06)
-        (xy 139.7 61.595)
+        (xy 143.764 99.06)
+        (xy 143.764 61.595)
         (xy 118.745 61.595)
       )

Commit message: Вариант с запресованной гайкой и обжатыми проводами
Parts:
- removed J17: A2, Connector_My:Coil
- removed J5: C2, Connector_My:Coil
- removed J7: B2, Connector_My:Coil
- J15, J18, J6: footprint Connector_My:Coil -> Connector_My:KFS2-M3
- moved J18 10.7 mm to (164.1, 67.3)
- moved J6 10.4 mm to (134.9, 67.3)
- moved J15 9.45 mm to (149.4, 55.4)
- moved J21 6.71 mm to (146.6, 90.7)
- moved J4 6.69 mm to (152.6, 90.7)
- moved J20 6.62 mm to (156.6, 90.7)
- moved J19 6.61 mm to (142.6, 90.7)
- moved H1 2.79 mm to (149.6, 95.5)
Routing:
- net GNDA: track 0.00 -> 21.6 mm, vias 0 -> 2
- net PTC_Coil_B: track 25.0 -> 24.0 mm, vias 0 -> 1
- net PTC_Coil_A: track 15.0 -> 16.0 mm, vias 0 -> 1
- removed copper zone on In2.Cu, net GNDA
Other:
- board size 58 x 58 mm -> 57.6 x 56.7 mm
