File: Плата обмоток/Плата обмоток.kicad_pcb (KiCad board)
At the start: 4 copper layers, 57.6 x 56.7 mm, 21 parts, among them J1 4900, J10 4900, J11 4900, J12 4900, J13 4900, J14 Conn_01x03, J15 C1, J16 4900, J18 B1, J19 B1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

Commit message: Добавил модель плты
Parts:
- J19, J20, J21, J4: footprint Connector_My:temp_wire -> Connector_My:temp_wire_2
- moved J20 9.53 mm to (150.9, 83.1)
- moved J19 8.58 mm to (146.6, 83.1)
- moved J21 7.81 mm to (148.3, 83.1)
- moved J4 7.62 mm to (152.7, 83.1)
- moved H1 0.76 mm to (149.6, 96.3)
Routing:
- net PTC_Coil_A: track 16.0 -> 21.1 mm, vias 1 -> 0
- net GNDA: track 21.6 -> 20.0 mm, vias 2 -> 1
- net PTC_Coil_B: track 24.0 -> 24.8 mm, vias 1 -> 0
Other:
- outline, holes or cut-outs redrawn

Commit message: Отправил на проверку в резонит
Parts:
- turned J6 to 180 degrees
Other:
- board text added: "A"
- board text added: "B"
- board text added: "C"
- board text added: "PTC"
Changed lines of the file:
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@@
 			(usegerberattributes yes)
 			(usegerberadvancedattributes yes)
-			(creategerberjobfile yes)
+			(creategerberjobfile no)
 			(dashed_line_dash_ratio 12.000000)
 			(dashed_line_gap_ratio 3.000000)
@@
 		(sheetname "Connectors")
 		(sheetfile "Connectors.kicad_sch")
+		(clearance 2)
 		(attr exclude_from_pos_files)
 		(fp_circle
@@
 		(sheetname "Connectors")
 		(sheetfile "Connectors.kicad_sch")
+		(clearance 2)
 		(attr exclude_from_pos_files)
 		(fp_circle
@@
 		(sheetname "Connectors")
 		(sheetfile "Connectors.kicad_sch")
+		(clearance 2)
 		(attr exclude_from_pos_files)
 		(fp_circle
@@
 		(model "/home/alexandr/Проекты/KAMAZ_Coil_PCB/3D модели/doc_2023-12-07_01-29-29.187 x .030 Quick-Fit terminal.STEP"
 			(offset
-				(xyz 2.5 -1.25 3.5)
+				(xyz 2.5 1.25 3.5)
 			)
 			(scale
@@
 			)
 			(rotate
-				(xyz 0 -180 0)
+				(xyz 0 -180 180)
 			)
 		)
@@
 		(model "/home/alexandr/Проекты/KAMAZ_Coil_PCB/3D модели/doc_2023-12-07_01-29-29.187 x .030 Quick-Fit terminal.STEP"
 			(offset
-				(xyz 2.5 -1.25 3.5)
+				(xyz 2.5 1.25 3.5)
 			)
 			(scale
@@
 			)
 			(rotate
-				(xyz 0 -180 0)
+				(xyz 0 -180 180)
 			)
 		)
@@
 		(model "/home/alexandr/Проекты/KAMAZ_Coil_PCB/3D модели/doc_2023-12-07_01-29-29.187 x .030 Quick-Fit terminal.STEP"
 			(offset
-				(xyz 2.5 -1.25 3.5)
+				(xyz 2.5 1.25 3.5)
 			)
 			(scale
@@
 			)
 			(rotate
-				(xyz 0 -180 0)
+				(xyz 0 -180 180)
 			)
 		)
@@
 		(model "/home/alexandr/Проекты/KAMAZ_Coil_PCB/3D модели/doc_2023-12-07_01-29-29.187 x .030 Quick-Fit terminal.STEP"
 			(offset
-				(xyz 2.5 -1.25 3.5)
+				(xyz 2.5 1.25 3.5)
 			)
 			(scale
@@
 			)
 			(rotate
-				(xyz 0 -180 0)
+				(xyz 0 -180 180)
 			)
 		)
@@
 		(model "/home/alexandr/Проекты/KAMAZ_Coil_PCB/3D модели/doc_2023-12-07_01-29-29.187 x .030 Quick-Fit terminal.STEP"
 			(offset
-				(xyz 2.5 -1.25 3.5)
+				(xyz 2.5 1.25 3.5)
 			)
 			(scale
@@
 			)
 			(rotate
-				(xyz 0 -180 0)
+				(xyz 0 -180 180)
 			)
 		)
@@
 			(at 0 0 180)
 			(size 7 7)
-			(drill 4.68)
+			(drill 4.22)
 			(layers "*.Cu" "*.Mask")
 			(remove_unused_layers no)
@@
 		(model "/home/alexandr/Проекты/KAMAZ_Coil_PCB/3D модели/KF2-M3-ET.stp"
 			(offset
-				(xyz 0 0 -3)
+				(xyz 0 0 1.5)
 			)
 			(scale
@@
 			)
 			(rotate
-				(xyz 0 -90 0)
+				(xyz 0 90 0)
 			)
 		)
@@
 	(footprint "Connector_My:KFS2-M3"
 		(layer "B.Cu")
-		(at 134.874 67.31 -90)
+		(at 134.874 67.31 180)
 		(property "Reference" "J6"
-			(at 0 6.556 90)
+			(at 0 6.556 0)
 			(unlocked yes)
 			(layer "B.SilkS")
@@
 		)
 		(property "Value" "A1"
-			(at 0 5.056 90)
+			(at 0 5.056 0)
 			(unlocked yes)
 			(layer "B.Fab")
@@
 		)
 		(property "Footprint" "Connector_My:KFS2-M3"
-			(at 0 0 90)
+			(at 0 0 360)
 			(layer "F.Fab")
 			(hide yes)
@@
 		)
 		(property "Datasheet" ""
-			(at 0 0 90)
+			(at 0 0 360)
 			(layer "F.Fab")
 			(hide yes)
@@
 		)
 		(property "Description" ""
-			(at 0 0 90)
+			(at 0 0 360)
 			(layer "F.Fab")
 			(hide yes)
@@
 		(attr through_hole)
 		(fp_text user "${REFERENCE}"
-			(at 0 3.556 90)
+			(at 0 3.556 0)
 			(unlocked yes)
 			(layer "B.Fab")
@@
 		)
 		(pad "1" thru_hole circle
-			(at 0 0 270)
+			(at 0 0 180)
 			(size 7 7)
-			(drill 4.68)
+			(drill 4.22)
 			(layers "*.Cu" "*.Mask")
 			(remove_unused_layers no)
@@
 		(model "/home/alexandr/Проекты/KAMAZ_Coil_PCB/3D модели/KF2-M3-ET.stp"
 			(offset
-				(xyz 0 0 -3)
+				(xyz 0 0 1.5)
 			)
 			(scale
@@
 			)
 			(rotate
-				(xyz 0 -90 0)
+				(xyz 0 90 0)
 			)
 		)
@@
 		(model "/home/alexandr/Проекты/KAMAZ_Coil_PCB/3D модели/doc_2023-12-07_01-29-29.187 x .030 Quick-Fit terminal.STEP"
 			(offset
-				(xyz 2.5 -1.25 3.5)
+				(xyz 2.5 1.25 3.5)
 			)
 			(scale
@@
 			)
 			(rotate
-				(xyz 0 -180 0)
+				(xyz 0 -180 180)
 			)
 		)
@@
 		(model "/home/alexandr/Проекты/KAMAZ_Coil_PCB/3D модели/doc_2023-12-07_01-29-29.187 x .030 Quick-Fit terminal.STEP"
 			(offset
-				(xyz 2.5 -1.25 3.5)
+				(xyz 2.5 1.25 3.5)
 			)
 			(scale
@@
 			)
 			(rotate
-				(xyz 0 -180 0)
+				(xyz 0 -180 180)
 			)
 		)
@@
 			(at 0 0 90)
 			(size 7 7)
-			(drill 4.68)
+			(drill 4.22)
 			(layers "*.Cu" "*.Mask")
 			(remove_unused_layers no)
@@
 		(model "/home/alexandr/Проекты/KAMAZ_Coil_PCB/3D модели/KF2-M3-ET.stp"
 			(offset
-				(xyz 0 0 -3)
+				(xyz 0 0 1.5)
 			)
 			(scale
@@
 			)
 			(rotate
-				(xyz 0 -90 0)
+				(xyz 0 90 0)
 			)
 		)
@@
 		(model "/home/alexandr/Проекты/KAMAZ_Coil_PCB/3D модели/doc_2023-12-07_01-29-29.187 x .030 Quick-Fit terminal.STEP"
 			(offset
-				(xyz 2.5 -1.25 3.5)
+				(xyz 2.5 1.25 3.5)
 			)
 			(scale
@@
 			)
 			(rotate
-				(xyz 0 -180 0)
+				(xyz 0 -180 180)
 			)
 		)
@@
 		(model "/home/alexandr/Проекты/KAMAZ_Coil_PCB/3D модели/doc_2023-12-07_01-29-29.187 x .030 Quick-Fit terminal.STEP"
 			(offset
-				(xyz 2.5 -1.25 3.5)
+				(xyz 2.5 1.25 3.5)
 			)
 			(scale
@@
 			)
 			(rotate
-				(xyz 0 -180 0)
+				(xyz 0 -180 180)
 			)
 		)
@@
 		(model "/home/alexandr/Проекты/KAMAZ_Coil_PCB/3D модели/doc_2023-12-07_01-29-29.187 x .030 Quick-Fit terminal.STEP"
 			(offset
-				(xyz 2.5 -1.25 3.5)
+				(xyz 2.5 1.25 3.5)
 			)
 			(scale
@@
 			)
 			(rotate
-				(xyz 0 -180 0)
+				(xyz 0 -180 180)
 			)
 		)
@@
 		(layer "Edge.Cuts")
 	)
+	(gr_text "PTC"
+		(at 152.4 92.456 0)
+		(layer "B.SilkS")
+		(effects
+			(font
+				(size 2 2)
+				(thickness 0.3)
+			)
+			(justify left bottom mirror)
+		)
+	)
+	(gr_text "A"
+		(at 165.608 74.93 0)
+		(layer "B.SilkS")
+		(effects
+			(font
+				(size 2 2)
+				(thickness 0.3)
+			)
+			(justify left bottom mirror)
+		)
+	)
+	(gr_text "B"
+		(at 150.368 61.722 0)
+		(layer "B.SilkS")
+		(effects
+			(font
+				(size 2 2)
+				(thickness 0.3)
+			)
+			(justify left bottom mirror)
+		)
+	)
+	(gr_text "C"
+		(at 136.398 74.93 0)
+		(layer "B.SilkS")
+		(effects
+			(font
+				(size 2 2)
+				(thickness 0.3)
+			)
+			(justify left bottom mirror)
+		)
+	)
 	(gr_text ""
