File: Плата обмоток/Connection List.kicad_sch (KiCad schematic)
At the start: 0 parts

Commit message: Изменения: добавил папку с отчетностью
Other:
- note removed: "1. Провода х распаиваются на плате в разъёмы J5, J6, J7, J15, J17, J18."
- note removed: "Датчик температуры C"
