File: Плата обмоток/Connectors.kicad_sch (KiCad schematic)
At the start: 22 parts, among them J1 4900, J10 4900, J11 4900, J12 4900, J13 4900, J14 A1, J15 A2, J16 B1, J17 B2, J18 C1, J19 C2, J2 4900, J3 4900, J4 Conn_01x02, J6 Conn_01x02, J7 Conn_01x02, J8 4900, J8 Conn_02x02_Odd_Even, J9 4900

Commit message: VER2.0
Parts:
- removed J4, J6, J7: Conn_01x02, Connector_Molex:Molex_PicoBlade_53048-0210_1x02_P1.25mm_Horizontal, symbol Connector_Generic:Conn_01x02
- removed J8: Conn_02x02_Odd_Even, Connector_PinSocket_2.54mm:PinSocket_2x02_P2.54mm_Vertical, symbol Connector_Generic:Conn_02x02_Odd_Even
- added J13: 4900, Connector_My:3551, symbol 4900:4900
- added J14: Conn_01x03, Connector_PinSocket_2.54mm:PinSocket_1x03_P2.54mm_Vertical, symbol Connector_Generic:Conn_01x03
- added J16 (x4): B1, Connector_My:temp_wire, symbol Connector:Conn_01x01_Pin
Connections:
- net GNDA: now also J14.3 (Pin_3), J16.1 (Pin_1), J16.1 (Pin_1)
- net PTC_Coil_A: now also J14.1 (Pin_1), J16.1 (Pin_1)
- net PTC_Coil_B: now also J14.2 (Pin_2), J16.1 (Pin_1)
- net A_OUT renamed A
- net B_OUT renamed B
- net B: now also J13.1, J13.2
- net C_OUT renamed C

Commit message: Вариант с запресованной гайкой и обжатыми проводами
Parts:
- removed J15: A2, Connector_My:Coil, symbol Connector:Conn_01x01_Pin
- removed J17: B2, Connector_My:Coil, symbol Connector:Conn_01x01_Pin
- removed J19: C2, Connector_My:Coil, symbol Connector:Conn_01x01_Pin
- J14, J16, J18: footprint Connector_My:Coil -> Connector_My:KFS2-M3
Other:
- moved on the sheet: J14, J16, J18
Changed lines of the file:
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@@
   (junction (at 194.31 105.41) (diameter 0) (color 0 0 0 0)
   )
-  (junction (at 207.01 68.58) (diameter 0) (color 0 0 0 0)
-  )
   (junction (at 212.09 124.46) (diameter 0) (color 0 0 0 0)
   )
@@
   (junction (at 212.09 132.08) (diameter 0) (color 0 0 0 0)
   )
-  (junction (at 185.42 68.58) (diameter 0) (color 0 0 0 0)
-  )
   (junction (at 212.09 105.41) (diameter 0) (color 0 0 0 0)
   )
   (junction (at 187.96 105.41) (diameter 0) (color 0 0 0 0)
   )
-  (junction (at 195.58 68.58) (diameter 0) (color 0 0 0 0)
-  )
   (junction (at 179.07 132.08) (diameter 0) (color 0 0 0 0)
   )
@@
     (stroke (width 0) (type default))
   )
-  (wire (pts (xy 182.88 68.58) (xy 185.42 68.58))
-    (stroke (width 0) (type default))
-  )
   (wire (pts (xy 212.09 125.73) (xy 213.36 125.73))
     (stroke (width 0) (type default))
@@
     (stroke (width 0) (type default))
   )
-  (wire (pts (xy 207.01 68.58) (xy 204.47 68.58))
-    (stroke (width 0) (type default))
-  )
   (wire (pts (xy 212.09 124.46) (xy 212.09 125.73))
     (stroke (width 0) (type default))
   )
-  (wire (pts (xy 198.12 66.04) (xy 198.12 68.58))
-    (stroke (width 0) (type default))
-  )
   (wire (pts (xy 179.07 125.73) (xy 179.07 124.46))
     (stroke (width 0) (type default))
@@
     (stroke (width 0) (type default))
   )
-  (wire (pts (xy 209.55 68.58) (xy 207.01 68.58))
-    (stroke (width 0) (type default))
-  )
   (wire (pts (xy 179.07 134.62) (xy 179.07 132.08))
     (stroke (width 0) (type default))
@@
     (stroke (width 0) (type default))
   )
-  (wire (pts (xy 207.01 68.58) (xy 207.01 69.85))
+  (wire (pts (xy 207.01 66.04) (xy 207.01 69.85))
     (stroke (width 0) (type default))
   )
@@
     (stroke (width 0) (type default))
   )
-  (wire (pts (xy 185.42 68.58) (xy 187.96 68.58))
-    (stroke (width 0) (type default))
-  )
   (wire (pts (xy 196.85 105.41) (xy 203.2 105.41))
     (stroke (width 0) (type default))
@@
     (stroke (width 0) (type default))
   )
-  (wire (pts (xy 193.04 68.58) (xy 193.04 66.04))
-    (stroke (width 0) (type default))
-  )
-  (wire (pts (xy 198.12 68.58) (xy 195.58 68.58))
-    (stroke (width 0) (type default))
-  )
-  (wire (pts (xy 195.58 68.58) (xy 195.58 69.85))
-    (stroke (width 0) (type default))
-  )
-  (wire (pts (xy 182.88 66.04) (xy 182.88 68.58))
-    (stroke (width 0) (type default))
-  )
-  (wire (pts (xy 187.96 68.58) (xy 187.96 66.04))
+  (wire (pts (xy 195.58 66.04) (xy 195.58 69.85))
     (stroke (width 0) (type default))
   )
@@
     (stroke (width 0) (type default))
   )
-  (wire (pts (xy 204.47 66.04) (xy 204.47 68.58))
-    (stroke (width 0) (type default))
-  )
   (wire (pts (xy 212.09 104.14) (xy 212.09 105.41))
     (stroke (width 0) (type default))
@@
     (stroke (width 0) (type default))
   )
-  (wire (pts (xy 195.58 68.58) (xy 193.04 68.58))
-    (stroke (width 0) (type default))
-  )
   (wire (pts (xy 203.2 105.41) (xy 203.2 104.14))
     (stroke (width 0) (type default))
   )
-  (wire (pts (xy 209.55 66.04) (xy 209.55 68.58))
-    (stroke (width 0) (type default))
-  )
-  (wire (pts (xy 185.42 68.58) (xy 185.42 69.85))
+  (wire (pts (xy 185.42 66.04) (xy 185.42 69.85))
     (stroke (width 0) (type default))
   )
@@
     )
   )
-  (symbol (lib_id "Connector:Conn_01x01_Pin") (at 209.55 60.96 270) (unit 1)
+  (symbol (lib_id "Connector:Conn_01x01_Pin") (at 207.01 60.96 270) (unit 1)
     (in_bom yes) (on_board yes) (dnp no)
-    (property "Reference" "J19" (at 209.55 59.69 90)
+    (property "Reference" "J14" (at 207.01 59.69 90)
       (effects (font (size 1.27 1.27)))
     )
-    (property "Value" "C2" (at 210.82 61.595 0)
-      (effects (font (size 1.27 1.27)) hide)
-    )
-    (property "Footprint" "Connector_My:Coil" (at 209.55 60.96 0)
-      (effects (font (size 1.27 1.27)) hide)
-    )
-    (property "Datasheet" "~" (at 209.55 60.96 0)
-      (effects (font (size 1.27 1.27)) hide)
-    )
-    (pin "1")
-    (instances
-      (project "Плата обмоток"
-        (path "/7abc0ce6-258d-434e-9c1a-83bc5738d31c"
-          (reference "J19") (unit 1)
-        )
-        (path "/7abc0ce6-258d-434e-9c1a-83bc5738d31c/b2a94a64-498f-4da2-994f-db948b492904"
-          (reference "J5") (unit 1)
-        )
-        (path "/7abc0ce6-258d-434e-9c1a-83bc5738d31c/c25d348d-11d7-47df-8e9d-61d215172e10"
-          (reference "J21") (unit 1)
-        )
-      )
-    )
-  )
-  (symbol (lib_id "Connector:Conn_01x01_Pin") (at 198.12 60.96 270) (unit 1)
-    (in_bom yes) (on_board yes) (dnp no)
-    (property "Reference" "J17" (at 198.12 59.69 90)
-      (effects (font (size 1.27 1.27)))
-    )
-    (property "Value" "B2" (at 199.39 61.595 0)
-      (effects (font (size 1.27 1.27)) hide)
-    )
-    (property "Footprint" "Connector_My:Coil" (at 198.12 60.96 0)
-      (effects (font (size 1.27 1.27)) hide)
-    )
-    (property "Datasheet" "~" (at 198.12 60.96 0)
-      (effects (font (size 1.27 1.27)) hide)
-    )
-    (pin "1")
-    (instances
-      (project "Плата обмоток"
-        (path "/7abc0ce6-258d-434e-9c1a-83bc5738d31c"
-          (reference "J17") (unit 1)
-        )
-        (path "/7abc0ce6-258d-434e-9c1a-83bc5738d31c/b2a94a64-498f-4da2-994f-db948b492904"
-          (reference "J7") (unit 1)
-        )
-        (path "/7abc0ce6-258d-434e-9c1a-83bc5738d31c/c25d348d-11d7-47df-8e9d-61d215172e10"
-          (reference "J23") (unit 1)
-        )
-      )
-    )
-  )
-  (symbol (lib_id "Connector:Conn_01x01_Pin") (at 204.47 60.96 270) (unit 1)
-    (in_bom yes) (on_board yes) (dnp no)
-    (property "Reference" "J14" (at 204.47 59.69 90)
-      (effects (font (size 1.27 1.27)))
-    )
-    (property "Value" "A1" (at 205.74 61.595 0)
-      (effects (font (size 1.27 1.27)) hide)
-    )
-    (property "Footprint" "Connector_My:Coil" (at 204.47 60.96 0)
-      (effects (font (size 1.27 1.27)) hide)
-    )
-    (property "Datasheet" "~" (at 204.47 60.96 0)
+    (property "Value" "A1" (at 208.28 61.595 0)
+      (effects (font (size 1.27 1.27)) hide)
+    )
+    (property "Footprint" "Connector_My:KFS2-M3" (at 207.01 60.96 0)
+      (effects (font (size 1.27 1.27)) hide)
+    )
+    (property "Datasheet" "~" (at 207.01 60.96 0)
       (effects (font (size 1.27 1.27)) hide)
     )
@@
     )
   )
-  (symbol (lib_id "Connector:Conn_01x01_Pin") (at 182.88 60.96 270) (unit 1)
+  (symbol (lib_id "Connector:Conn_01x01_Pin") (at 185.42 60.96 270) (unit 1)
     (in_bom yes) (on_board yes) (dnp no)
-    (property "Reference" "J16" (at 182.88 59.69 90)
+    (property "Reference" "J16" (at 185.42 59.69 90)
       (effects (font (size 1.27 1.27)))
     )
-    (property "Value" "B1" (at 184.15 61.595 0)
-      (effects (font (size 1.27 1.27)) hide)
-    )
-    (property "Footprint" "Connector_My:Coil" (at 182.88 60.96 0)
-      (effects (font (size 1.27 1.27)) hide)
-    )
-    (property "Datasheet" "~" (at 182.88 60.96 0)
+    (property "Value" "B1" (at 186.69 61.595 0)
+      (effects (font (size 1.27 1.27)) hide)
+    )
+    (property "Footprint" "Connector_My:KFS2-M3" (at 185.42 60.96 0)
+      (effects (font (size 1.27 1.27)) hide)
+    )
+    (property "Datasheet" "~" (at 185.42 60.96 0)
       (effects (font (size 1.27 1.27)) hide)
     )
@@
     )
   )
-  (symbol (lib_id "Connector:Conn_01x01_Pin") (at 193.04 60.96 270) (unit 1)
+  (symbol (lib_id "Connector:Conn_01x01_Pin") (at 195.58 60.96 270) (unit 1)
     (in_bom yes) (on_board yes) (dnp no)
-    (property "Reference" "J18" (at 193.04 59.69 90)
+    (property "Reference" "J18" (at 195.58 59.69 90)
       (effects (font (size 1.27 1.27)))
     )
-    (property "Value" "C1" (at 194.31 61.595 0)
-      (effects (font (size 1.27 1.27)) hide)
-    )
-    (property "Footprint" "Connector_My:Coil" (at 193.04 60.96 0)
-      (effects (font (size 1.27 1.27)) hide)
-    )
-    (property "Datasheet" "~" (at 193.04 60.96 0)
+    (property "Value" "C1" (at 196.85 61.595 0)
+      (effects (font (size 1.27 1.27)) hide)
+    )
+    (property "Footprint" "Connector_My:KFS2-M3" (at 195.58 60.96 0)
+      (effects (font (size 1.27 1.27)) hide)
+    )
+    (property "Datasheet" "~" (at 195.58 60.96 0)
       (effects (font (size 1.27 1.27)) hide)
     )
@@
         )
       )
-    )
-  )
-  (symbol (lib_id "Connector:Conn_01x01_Pin") (at 187.96 60.96 270) (unit 1)
-    (in_bom yes) (on_board yes) (dnp no)
-    (property "Reference" "J15" (at 187.96 59.69 90)
-      (effects (font (size 1.27 1.27)))
-    )
-    (property "Value" "A2" (at 189.23 61.595 0)
-      (effects (font (size 1.27 1.27)) hide)
-    )
-    (property "Footprint" "Connector_My:Coil" (at 187.96 60.96 0)
-      (effects (font (size 1.27 1.27)) hide)
-    )
-    (property "Datasheet" "~" (at 187.96 60.96 0)
-      (effects (font (size 1.27 1.27)) hide)
-    )
-    (pin "1")
-    (instances
-      (project "Плата обмоток"
-        (path "/7abc0ce6-258d-434e-9c1a-83bc5738d31c"
-          (reference "J15") (unit 1)
-        )
-        (path "/7abc0ce6-258d-434e-9c1a-83bc5738d31c/b2a94a64-498f-4da2-994f-db948b492904"
-          (reference "J17") (unit 1)
-        )
-        (path "/7abc0ce6-258d-434e-9c1a-83bc5738d31c/c25d348d-11d7-47df-8e9d-61d215172e10"
-          (reference "J27") (unit 1)
-        )
-      )

Commit message: Добавил модель плты
Parts:
- renumbered H2 to H1, H3 to H2, H4 to H3, J12 to J10, J3 to J11, J10 to J12, J18 to J15, J13 to J16, J16 to J18, J16 to J19, J8 to J2, J16 to J20, J16 to J21, J11 to J3, J16 to J4, J14 to J6, J2 to J8
